Commit message: 0629 config urdf

File: src/roma_car/urdf/roma_car.urdf (robot description, URDF)
Before this commit: robot roma_car, 11 links, 10 joints
Joints:
- joint LB_drive_joint: limit lower=0 upper=0 effort=0 velocity=0 -> lower=0 upper=0 effort=1.6 velocity=1000
- joint LB_susp_joint: limit lower=0 upper=0.5 effort=0 velocity=0 -> lower=-0.03 upper=0.03 effort=1 velocity=1
- joint LF_drive_joint: limit lower=0 upper=0 effort=0 velocity=0 -> lower=0 upper=0 effort=1.6 velocity=1000
- joint LF_steer_joint: limit lower=0 upper=0 effort=0 velocity=0 -> lower=-0.68 upper=0.68 effort=3.0 velocity=5.0
- joint LF_susp_joint: limit lower=0 upper=0.5 effort=0 velocity=0 -> lower=-0.03 upper=0.03 effort=1 velocity=1
- joint RB_drive_joint: limit lower=0 upper=0 effort=0 velocity=0 -> lower=0 upper=0 effort=1.6 velocity=1000
- joint RB_susp_joint: limit lower=0 upper=0.5 effort=0 velocity=0 -> lower=-0.03 upper=0.03 effort=1 velocity=1
- joint RF_drive_joint: limit lower=0 upper=0 effort=0 velocity=0 -> lower=0 upper=0 effort=1.6 velocity=1000
- joint RF_steer_joint: limit lower=0 upper=0 effort=0 velocity=0 -> lower=-0.68 upper=0.68 effort=3.0 velocity=5.0
- joint RF_susp_joint: limit lower=0 upper=0.5 effort=0 velocity=0 -> lower=-0.03 upper=0.03 effort=1 velocity=1

Commit message: 0812 add urdf file

File: src/roma_car/urdf/roma_car.urdf (robot description, URDF)
Before this commit: robot roma_car, 11 links, 10 joints
Joints:
- joint LF_drive_joint: axis 0 -0.999999999999973 0 -> 0 -1 0; parent LF_steer_link -> LF_susp_link
- joint LF_steer_joint: origin xyz=0 0 0 rpy=0 0 0 -> xyz=0.202 0.14049 0.0274 rpy=0 0 0; parent LF_susp_link -> base_link
- joint LF_susp_joint: origin xyz=0.202 0.14049 0.0274 rpy=0 0 0 -> xyz=0 0 0 rpy=0 0 0; parent base_link -> LF_steer_link
- joint RF_drive_joint: parent RF_steer_link -> RF_susp_link
- joint RF_steer_joint: origin xyz=0 0 0 rpy=0 0 0 -> xyz=0.202 -0.1401 0.024747 rpy=0 0 0; parent RF_susp_link -> base_link
- joint RF_susp_joint: origin xyz=0.202 -0.1401 0.024747 rpy=0 0 0 -> xyz=0 0 0 rpy=0 0 0; parent base_link -> RF_steer_link
